Commit message: add visualizations for pointclouds

File: collision_avoidance_example/xarm7_gripper_urdf/xarm7_with_gripper.urdf (robot description, URDF)
Before this commit: robot UF_ROBOT, 18 links, 17 joints
Links:
- link link_base: geometry collision mesh filename=xarm_description/meshes/xarm7/collision/link0.obj; visual mesh filename=xarm_description/meshes/xarm7/visual/link0.stl

File: collision_avoidance_example/xarm7_urdf/xarm7_robot.urdf (robot description, URDF)
Before this commit: robot UF_ROBOT, 10 links, 9 joints
Links:
- removed link link_base
- added link link0, mass 0.88556; collision mesh filename=package://xarm_description/meshes/xarm7/collision/link0.obj; visual mesh filename=package://xarm_description/meshes/xarm7/visual/link0.stl
Joints:
- joint joint1: parent link_base -> link0
- joint world_joint: child link_base -> link0
